File: BLDC.sch (KiCad schematic (older format))
At the start: 162 parts, among them J1 436500513, J2 436500313, J3 TC2030-MCP-NL, J4 436500513, Q0 2N7002A-7, Q1 2N7002A-7, U0 LSM6DS3US, U1 LM5008, U10 OPA365, U11 OPA365, U12 MCP9808, U13 AS5047D-ATSM, U2 LM5166, U3 TLV702, U4 TLV702, U5 DRV8312, U6 ISL32458E, U7 SN74LVC1G66DCKR, U8 OPA365, U9 STM32F405RG

Commit message: First draft of rework, major changes to placement, routing and components choice
Parts:
- removed C10, C4, C6: 1.0nF, RS485-tester-STM32F405RG.place.kicad:CAPC1005X55, symbol BLDC-rescue:capacitor-sym$2-BLDC-rescue
- removed C17, C41: 100.0nF, RS485-tester-STM32F405RG.place.kicad:CAPC3216X160, symbol BLDC-rescue:capacitor-sym$2$1-BLDC-rescue
- removed C28: 4.7μF, RS485-tester-STM32F405RG.place.kicad:CAPC3216X160, symbol BLDC-rescue:capacitor-sym$2$1-BLDC-rescue
- removed C29, C3, C34: 100.0nF, RS485-tester-STM32F405RG.place.kicad:CAPC1005X55, symbol BLDC-rescue:capacitor-sym$2-BLDC-rescue
- removed C31: 22.0μF, RS485-tester-STM32F405RG.place.kicad:CAPC3216X160, symbol BLDC-rescue:capacitor-sym$2$1-BLDC-rescue
- removed C33, C44, C5, C8: 1.0μF, RS485-tester-STM32F405RG.place.kicad:CAPC1005X55, symbol BLDC-rescue:capacitor-sym$2-BLDC-rescue
- removed C45: 1.0μF, RS485-tester-STM32F405RG.place.kicad:CAPC3216X160, symbol BLDC-rescue:capacitor-sym$2$1-BLDC-rescue
- removed C59: 1.0μF, RS485-tester-STM32F405RG.place.kicad:CAPC1005X55, symbol BLDC-rescue:capacitor-sym$2$1-BLDC-rescue
- removed C65: 4.7nF, RS485-tester-STM32F405RG.place.kicad:CAPC1005X55, symbol BLDC-rescue:capacitor-sym$2-BLDC-rescue
- removed C70, C71, C72: DNP, RS485-tester-STM32F405RG.place.kicad:CAPC1005X55, symbol BLDC-rescue:capacitor-sym$2-BLDC-rescue
- removed C9: 10.0nF, RS485-tester-STM32F405RG.place.kicad:CAPC1005X55, symbol BLDC-rescue:capacitor-sym$2-BLDC-rescue
- removed D1: DFLS1100, RS485-tester-STM32F405RG.place.kicad:DFLS1100-fp, symbol BLDC-rescue:diode-sym-BLDC-rescue
- removed L1: 330.0μH, RS485-tester-STM32F405RG.place.kicad:coilcraft-LPS4018-334MRB, symbol BLDC-rescue:inductor-sym$1-BLDC-rescue
- removed Q0, Q1: 2N7002A-7, RS485-tester-STM32F405RG.place.kicad:SOT95P280X100-3N, symbol BLDC-rescue:fet-sym-BLDC-rescue
- removed R1: 680.0mΩ, RS485-tester-STM32F405RG.place.kicad:RESC1005X35, symbol BLDC-rescue:resistor-sym$1-BLDC-rescue
- removed R11: MMZ1005Y152CT000, RS485-tester-STM32F405RG.place.kicad:RESC1005X35, symbol BLDC-rescue:resistor-sym$1-BLDC-rescue
- removed R12: 2.67kΩ, RS485-tester-STM32F405RG.place.kicad:RESC1005X35, symbol BLDC-rescue:resistor-sym-BLDC-rescue
- removed R13, R40, R58: 5.49kΩ, RS485-tester-STM32F405RG.place.kicad:RESC1005X35, symbol BLDC-rescue:resistor-sym$1-BLDC-rescue
- removed R14, R26: 100.0kΩ, RS485-tester-STM32F405RG.place.kicad:RESC1005X35, symbol BLDC-rescue:resistor-sym-BLDC-rescue
- removed R16, R24, R45, R46, R53, R59: 100Ω, RS485-tester-STM32F405RG.place.kicad:RESC1005X35, symbol BLDC-rescue:resistor-sym-BLDC-rescue
- removed R18: 301.0kΩ, RS485-tester-STM32F405RG.place.kicad:RESC1005X35, symbol BLDC-rescue:resistor-sym-BLDC-rescue
- removed R20, R23, R51: 9.53kΩ, RS485-tester-STM32F405RG.place.kicad:RESC1005X35, symbol BLDC-rescue:resistor-sym$1-BLDC-rescue
- removed R22, R44, R54: 10.0kΩ, RS485-tester-STM32F405RG.place.kicad:RESC1005X35, symbol BLDC-rescue:resistor-sym-BLDC-rescue
- removed R28: 137.0kΩ, RS485-tester-STM32F405RG.place.kicad:RESC1005X35, symbol BLDC-rescue:resistor-sym-BLDC-rescue
- removed R29: 2.7Ω, RS485-tester-STM32F405RG.place.kicad:RESC1005X35, symbol BLDC-rescue:resistor-sym-BLDC-rescue
- removed R34: 9.76MΩ, RS485-tester-STM32F405RG.place.kicad:RESC1608X45, symbol BLDC-rescue:resistor-sym-BLDC-rescue
- removed R35, R37, R42: CRA2512-FZ-R010ELF, RS485-tester-STM32F405RG.place.kicad:RESC6332X35, symbol BLDC-rescue:resistor-sym$2-BLDC-rescue
- removed R36, R7: 28.7kΩ, RS485-tester-STM32F405RG.place.kicad:RESC1005X35, symbol BLDC-rescue:resistor-sym-BLDC-rescue
- removed R41: 866.0kΩ, RS485-tester-STM32F405RG.place.kicad:RESC1005X35, symbol BLDC-rescue:resistor-sym-BLDC-rescue
- removed R49, R60, R8: 4.3kΩ, RS485-tester-STM32F405RG.place.kicad:RESC1005X35, symbol BLDC-rescue:resistor-sym$1-BLDC-rescue
- removed U1: LM5008, RS485-tester-STM32F405RG.place.kicad:VSSOP-8, symbol BLDC-rescue:ti-LM5008-BLDC-rescue
- removed U10, U11, U8: OPA365, RS485-tester-STM32F405RG.place.kicad:SOT95P280X145-5N, symbol BLDC-rescue:ti-OPA365-BLDC-rescue
- removed U4: TLV702, RS485-tester-STM32F405RG.place.kicad:SOT95P280X145-5N, symbol BLDC-rescue:ti-TLV702-BLDC-rescue
- added C10: 4.1pF, Capacitor_SMD:C_0402_1005Metric, symbol Device:C_Small
- added C11: 150pF, Capacitor_SMD:C_0805_2012Metric, symbol Device:C_Small
- added C12, C17: 4.7μF, Capacitor_SMD:C_1206_3216Metric, symbol Device:C_Small
- added C13, C14, C16: 100.0nF, Capacitor_SMD:C_0603_1608Metric, symbol Device:C_Small
- added C3, C5: 2.2uF, Capacitor_SMD:C_1206_3216Metric, symbol Device:C_Small
- added C4: 2.2μF, Capacitor_SMD:C_1210_3225Metric, symbol Device:C_Small
- added C6, C7: 100.0μF, Capacitor_SMD:C_1206_3216Metric, symbol Device:C_Small
- added C8: 56.0nF, Capacitor_SMD:C_0402_1005Metric, symbol Device:C_Small
- added L2: 220μH, Inductor_SMD:L_6.3x6.3_H3, symbol BLDC:inductor-sym
- added R1: 196.0kΩ, Resistor_SMD:R_0402_1005Metric, symbol Device:R_Small_US
- added R11: 124.0kΩ, Resistor_SMD:R_0402_1005Metric, symbol Device:R_Small_US
- added R7: 8.87MΩ, Resistor_SMD:R_0805_2012Metric, symbol Device:R_Small_US
- added R8: 1.1MΩ, Resistor_SMD:R_0402_1005Metric, symbol Device:R_Small_US
- added U17, U18, U19: INA250, Package_SO:TSSOP-16_4.4x5mm_P0.65mm, symbol BLDC:INA250
- added U4: LM5166, Package_SON:VSON-10-1EP_3x3mm_P0.5mm_EP1.65x2.4mm_ThermalVias, symbol BLDC:ti-LM5166
- added U8: ADP7142AUJZ-3.3, Package_TO_SOT_SMD:TSOT-23-5, symbol Regulator_Linear:ADP7142AUJZ-3.3
- C1: footprint RS485-tester-STM32F405RG.place.kicad:CAPC3216X160 -> Capacitor_SMD:C_0805_2012Metric; symbol BLDC-rescue:capacitor-sym$2$1-BLDC-rescue -> Device:C_Small
- C15, C18, C19, C2, C20, C21, C24, C26, C27, C30, C32, C36, C38, C39, C40, C42, C43, C46, C47, C48, C49, C50, C53, C54, C56, C57, C60, C61, C62, C63, C66, C67, C73: footprint RS485-tester-STM32F405RG.place.kicad:CAPC1005X55 -> Capacitor_SMD:C_0402_1005Metric; symbol BLDC-rescue:capacitor-sym$2-BLDC-rescue -> Device:C_Small
- C22, C25, C69: symbol BLDC-rescue:capacitor-sym$1-BLDC-rescue -> Device:CP_Small
- C23, C52: footprint RS485-tester-STM32F405RG.place.kicad:CAPC1005X55 -> Capacitor_SMD:C_0402_1005Metric; symbol BLDC-rescue:capacitor-sym$2$1-BLDC-rescue -> Device:C_Small
- C35, C51: symbol BLDC-rescue:capacitor-sym$2$1-BLDC-rescue -> Device:C_Small
- C37: footprint RS485-tester-STM32F405RG.place.kicad:CAPC3216X160 -> Capacitor_SMD:C_0402_1005Metric; symbol BLDC-rescue:capacitor-sym$2-BLDC-rescue -> Device:C_Small; Maximum Voltage 50.0V -> 16.0V
- C58: value 47.0μF -> 100.0μF; footprint RS485-tester-STM32F405RG.place.kicad:CAPC3216X160 -> Capacitor_SMD:C_1206_3216Metric; symbol BLDC-rescue:capacitor-sym$2$1-BLDC-rescue -> Device:C_Small; Capacitance 47.0uF -> 100.0uF; Maximum Voltage 10.0V -> 6.3V
- C64, C68: footprint RS485-tester-STM32F405RG.place.kicad:CAPC3216X160 -> Capacitor_SMD:C_0805_2012Metric; symbol BLDC-rescue:capacitor-sym$2-BLDC-rescue -> Device:C_Small
- D0, D2: symbol BLDC-rescue:diode-sym$2-BLDC-rescue -> BLDC:diode-sym$2
- D3: symbol BLDC-rescue:rhom-SMLP34RGB-BLDC-rescue -> BLDC:rhom-SMLP34RGB
- H0, H1, H2, H3: symbol BLDC-rescue:hole-sym-BLDC-rescue -> BLDC:hole-sym
- J1, J4: symbol BLDC-rescue:microfit-5-BLDC-rescue -> BLDC:microfit-5
- J2: symbol BLDC-rescue:generic-box-sym$2-BLDC-rescue -> BLDC:generic-box-sym$2
- J3: symbol BLDC-rescue:TC2030-MCP-NL-BLDC-rescue -> BLDC:TC2030-MCP-NL
- L0: value 150.0μH -> 22.0μH; footprint RS485-tester-STM32F405RG.place.kicad:coilcraft-CLF6045-fp -> Inductor_SMD:L_7.3x7.3_H4.5; symbol BLDC-rescue:inductor-sym-BLDC-rescue -> BLDC:inductor-sym; Inductance 150.0uH -> 22.0uH; Maximum Current 0.2A -> 2A
- R0, R10, R15, R17, R19, R2, R21, R27, R3, R30, R31, R33, R38, R39, R4, R43, R47, R48, R50, R52, R55, R56, R6, R61, R62, R63, R64, R9: footprint RS485-tester-STM32F405RG.place.kicad:RESC1005X35 -> Resistor_SMD:R_0402_1005Metric; symbol BLDC-rescue:resistor-sym-BLDC-rescue -> Device:R_Small_US
- R25: value 301.0kΩ -> 271.0kΩ; footprint RS485-tester-STM32F405RG.place.kicad:RESC1005X35 -> Resistor_SMD:R_0402_1005Metric; symbol BLDC-rescue:resistor-sym-BLDC-rescue -> Device:R_Small_US; Resistance 301000.0ohm -> 271000.0ohm; Tolerance 2.0% -> 0.1%
- R32: value MMZ1005Y152CT000 -> TBC; footprint RS485-tester-STM32F405RG.place.kicad:RESC1005X35 -> Resistor_SMD:R_0805_2012Metric; symbol BLDC-rescue:resistor-sym$1-BLDC-rescue -> Device:R_Small_US; Maximum Power 0.0625W -> 0.25W
- R5: value 137.0kΩ -> 124.0kΩ; footprint RS485-tester-STM32F405RG.place.kicad:RESC1005X35 -> Resistor_SMD:R_0402_1005Metric; symbol BLDC-rescue:resistor-sym-BLDC-rescue -> Device:R_Small_US; Resistance 137000.0ohm -> 124000.0ohm; Tolerance 2.0% -> 0.1%
- S1: symbol BLDC-rescue:omron-B3U-1000P-BLDC-rescue -> BLDC:omron-B3U-1000P
- U0: symbol BLDC-rescue:st-LSM6DS3US-BLDC-rescue -> BLDC:st-LSM6DS3US
- U12: symbol BLDC-rescue:mcp-MCP9808-BLDC-rescue -> BLDC:mcp-MCP9808
- U13: symbol BLDC-rescue:ams-as50487d-BLDC-rescue -> BLDC:ams-as50487d
- U2: footprint RS485-tester-STM32F405RG.place.kicad:VSON-10 -> Package_SON:VSON-10-1EP_3x3mm_P0.5mm_EP1.65x2.4mm_ThermalVias; symbol BLDC-rescue:ti-LM5166-BLDC-rescue -> BLDC:ti-LM5166
- U3: symbol BLDC-rescue:ti-TLV702-BLDC-rescue -> BLDC:ti-TLV702
- U5: symbol BLDC-rescue:st-DRV8312-BLDC-rescue -> BLDC:st-DRV8312
- U6: symbol BLDC-rescue:isl-ISL32459E-BLDC-rescue -> BLDC:isl-ISL32459E
- U7: symbol BLDC-rescue:SN74LVC1G66DCKR-BLDC-rescue -> BLDC:SN74LVC1G66DCKR
- U9: symbol BLDC-rescue:stmicro-STM32F405RG-BLDC-rescue -> BLDC:stmicro-STM32F405RG
- XTAL0: symbol BLDC-rescue:crystal-sym-BLDC-rescue -> BLDC:crystal-sym
Connections:
- net labels removed: 12v0_EN, pi_reg-3v3_reg-3v9_en
- wire segments 599 -> 512
Other:
- moved on the sheet: C51

Commit message: Breaking changes, changed IO pin assigment of STM32 to simplify routing, various optimizations
Parts:
- removed C23: 10.0nF, Capacitor_SMD:C_0402_1005Metric, symbol Device:C_Small
- removed C3, C5: 2.2uF, Capacitor_SMD:C_1206_3216Metric, symbol Device:C_Small
- removed R17: 3.3Ω, Resistor_SMD:R_0402_1005Metric, symbol Device:R_Small_US
- removed U8: ADP7142AUJZ-3.3, Package_TO_SOT_SMD:TSOT-23-5, symbol Regulator_Linear:ADP7142AUJZ-3.3
- C21: value 1.0μF -> 100nF
- U12: footprint RS485-tester-STM32F405RG.place.kicad:VSSOP-8 -> RS485-tester-STM32F405RG.place.kicad:MSOP-8
Connections:
- net labels removed: +3.3VA
- wire segments 512 -> 491
Other:
- moved on the sheet: C27

Commit message: Cleared DRC errors, changed minimum track width to 6 mil for cheaper manufacturing.
Parts:
- removed C22, C69: 220uF, RS485-tester-STM32F405RG.place.kicad:CAPAE12500X13500, symbol Device:CP_Small
- added C3, C5: 180uF, Capacitor_THT:CP_Radial_D8.0mm_P3.50mm, symbol Device:CP_Small
- C25: value 220uF -> 180uF; footprint RS485-tester-STM32F405RG.place.kicad:CAPAE12500X13500 -> Capacitor_THT:CP_Radial_D8.0mm_P3.50mm; Capacitance 220.0uF -> 180.0uF
- U9: footprint RS485-tester-STM32F405RG.place.kicad:LQFP64 -> Package_QFP:LQFP-64_10x10mm_P0.5mm
Connections:
- net +48V: now also C3.1, C5.1
- net ENC_MAG_LO: now also U9.35 (PB14); no longer U9.38 (PC7)
- net GND: now also C3.2, C5.2
- net MOT_RST_A: now also U9.38 (PC7); no longer U9.35 (PB14)
Changed lines of the file:
@@
 Text Label 11450 5750 1    40   ~ 0
 SPI_CS
-Text Label 11950 7250 0    40   ~ 0
+Text Label 11950 6950 0    40   ~ 0
 MOT_RST_A
 Text Label 9750 6550 2    40   ~ 0
@@
 Text Label 11950 7050 0    40   ~ 0
 ENC_MAG_HI
-Text Label 11950 6950 0    40   ~ 0
+Text Label 11950 7250 0    40   ~ 0
 ENC_MAG_LO
 Wire Wire Line
@@
 $EndComp
 $Comp
-L Device:CP_Small C69
-U 1 1 5B522179
-P 1950 3300
-F 0 "C69" H 2050 3350 28  0000 L CNN
-F 1 "220uF" H 2050 3300 28  0000 L CNN
-F 2 "RS485-tester-STM32F405RG.place.kicad:CAPAE12500X13500" H 1950 3300 60  0001 C CNN
-F 3 "" H 1950 3300 60  0001 C CNN
-F 4 "220.0uF" H 1950 3300 60  0001 C CNN "Capacitance"
-F 5 "20.0%" H 1950 3300 60  0001 C CNN "Tolerance"
-F 6 "63.0V" H 2050 3250 28  0000 L CNN "Maximum Voltage"
-	1    1950 3300
-	1    0    0    -1
-$EndComp
-$Comp
 L Device:C_Small C68
 U 1 1 5B48C3F2
@@
 F 0 "U9" H 11850 7600 28  0000 L CNN
 F 1 "STM32F405RG" H 11600 5800 28  0000 L CNN
-F 2 "RS485-tester-STM32F405RG.place.kicad:LQFP64" H 10850 6700 60  0001 C CNN
+F 2 "Package_QFP:LQFP-64_10x10mm_P0.5mm" H 10850 6700 60  0001 C CNN
 F 3 "" H 10850 6700 60  0001 C CNN
 	1    10850 6700
@@
 P 1250 3300
 F 0 "C25" H 1350 3350 28  0000 L CNN
-F 1 "220uF" H 1350 3300 28  0000 L CNN
-F 2 "RS485-tester-STM32F405RG.place.kicad:CAPAE12500X13500" H 1250 3300 60  0001 C CNN
+F 1 "180uF" H 1350 3300 28  0000 L CNN
+F 2 "Capacitor_THT:CP_Radial_D8.0mm_P3.50mm" H 1250 3300 60  0001 C CNN
 F 3 "" H 1250 3300 60  0001 C CNN
-F 4 "220.0uF" H 1250 3300 60  0001 C CNN "Capacitance"
+F 4 "180.0uF" H 1250 3300 60  0001 C CNN "Capacitance"
 F 5 "20.0%" H 1250 3300 60  0001 C CNN "Tolerance"
 F 6 "63.0V" H 1350 3250 28  0000 L CNN "Maximum Voltage"
@@
 $EndComp
 $Comp
-L Device:CP_Small C22
-U 1 1 5B48C451
-P 1600 3300
-F 0 "C22" H 1700 3350 28  0000 L CNN
-F 1 "220uF" H 1700 3300 28  0000 L CNN
-F 2 "RS485-tester-STM32F405RG.place.kicad:CAPAE12500X13500" H 1600 3300 60  0001 C CNN
-F 3 "" H 1600 3300 60  0001 C CNN
-F 4 "220.0uF" H 1600 3300 60  0001 C CNN "Capacitance"
-F 5 "20.0%" H 1600 3300 60  0001 C CNN "Tolerance"
-F 6 "63.0V" H 1700 3250 28  0000 L CNN "Maximum Voltage"
-	1    1600 3300
-	1    0    0    -1
-$EndComp
-$Comp
 L Device:R_Small_US R21
 U 1 1 5B48C450
@@
 Wire Wire Line
 	10500 8050 10500 8200
+$Comp
+L Device:CP_Small C3
+U 1 1 5D438A97
+P 1600 3300
+F 0 "C3" H 1700 3350 28  0000 L CNN
+F 1 "180uF" H 1700 3300 28  0000 L CNN
+F 2 "Capacitor_THT:CP_Radial_D8.0mm_P3.50mm" H 1600 3300 60  0001 C CNN
+F 3 "" H 1600 3300 60  0001 C CNN
+F 4 "180.0uF" H 1600 3300 60  0001 C CNN "Capacitance"
+F 5 "20.0%" H 1600 3300 60  0001 C CNN "Tolerance"
+F 6 "63.0V" H 1700 3250 28  0000 L CNN "Maximum Voltage"
+	1    1600 3300
+	1    0    0    -1
+$EndComp
+$Comp
+L Device:CP_Small C5
+U 1 1 5D43A18E
+P 1950 3300
+F 0 "C5" H 2050 3350 28  0000 L CNN
+F 1 "180uF" H 2050 3300 28  0000 L CNN
+F 2 "Capacitor_THT:CP_Radial_D8.0mm_P3.50mm" H 1950 3300 60  0001 C CNN
+F 3 "" H 1950 3300 60  0001 C CNN
+F 4 "180.0uF" H 1950 3300 60  0001 C CNN "Capacitance"
+F 5 "20.0%" H 1950 3300 60  0001 C CNN "Tolerance"
+F 6 "63.0V" H 2050 3250 28  0000 L CNN "Maximum Voltage"
+	1    1950 3300
+	1    0    0    -1
+$EndComp
 $EndSCHEMATC

Commit message: Removed capacitor that would be in contact in 3d mounting, fixed silkscreen
Parts:
- removed C5: 180uF, Capacitor_THT:CP_Radial_D8.0mm_P3.50mm, symbol Device:CP_Small
Changed lines of the file:
@@
 Wire Wire Line
 	9500 5250 9500 5350
-Wire Wire Line
-	1950 3550 1950 3400
 Connection ~ 1600 3550
 Wire Wire Line
@@
 	1600 2850 1600 3200
 Connection ~ 1250 2850
-Wire Wire Line
-	1950 2850 1950 3200
 Connection ~ 1600 2850
 Connection ~ 9450 7150
@@
 Wire Wire Line
 	2300 3550 2300 3500
-Connection ~ 1950 3550
 Wire Wire Line
 	2300 2850 2300 2900
-Connection ~ 1950 2850
 Wire Wire Line
 	10250 8050 10500 8050
@@
 	1600 3550 1600 3650
 Wire Wire Line
-	1600 3550 1950 3550
-Wire Wire Line
 	1250 3550 1600 3550
 Wire Wire Line
 	1250 2850 1600 2850
 Wire Wire Line
-	1600 2850 1950 2850
-Wire Wire Line
 	9450 7150 9750 7150
 Wire Wire Line
@@
 	1100 9000 1250 9000
 Wire Wire Line
-	1950 3550 2300 3550
-Wire Wire Line
-	1950 2850 2300 2850
-Wire Wire Line
 	900  2100 900  2200
 Wire Wire Line
@@
 	1    0    0    -1
 $EndComp
-$Comp
-L Device:CP_Small C5
-U 1 1 5D43A18E
-P 1950 3300
-F 0 "C5" H 2050 3350 28  0000 L CNN
-F 1 "180uF" H 2050 3300 28  0000 L CNN
-F 2 "Capacitor_THT:CP_Radial_D8.0mm_P3.50mm" H 1950 3300 60  0001 C CNN
-F 3 "" H 1950 3300 60  0001 C CNN
-F 4 "180.0uF" H 1950 3300 60  0001 C CNN "Capacitance"
-F 5 "20.0%" H 1950 3300 60  0001 C CNN "Tolerance"
-F 6 "63.0V" H 2050 3250 28  0000 L CNN "Maximum Voltage"
-	1    1950 3300
-	1    0    0    -1
-$EndComp
+Wire Wire Line
+	1600 3550 2300 3550
+Wire Wire Line
+	1600 2850 2300 2850
 $EndSCHEMATC

Commit message: WIP changed capacitors back to SMT
Parts:
- removed C43: 1.0μF, Capacitor_SMD:C_0402_1005Metric, symbol Device:C_Small
- added C22, C5, C9: 180uF, Capacitor_SMD:CP_Elec_10x10, symbol Device:CP_Small
- added C23, C28: 150pF, Capacitor_SMD:C_0805_2012Metric, symbol Device:C_Small
- added R12, R13: 8.87MΩ, Resistor_SMD:R_0805_2012Metric, symbol Device:R_Small_US
- C25, C3: footprint Capacitor_THT:CP_Radial_D8.0mm_P3.50mm -> Capacitor_SMD:CP_Elec_10x10
- C35: footprint RS485-tester-STM32F405RG.place.kicad:CAPC3216X160 -> Capacitor_SMD:C_0805_2012Metric
Connections:
- net +48V: now also C22.1, C5.1, C9.1
- net GND: now also C22.2, C23.1, C28.1, C5.2, C9.2
- new net: C23.2, R12.1
- new net IN: C28.2, R12.2, R13.1, R13.2
Other:
- moved on the sheet: C39

Commit message: Fixed DRC errors, added ground pour, fixed courtyards of connectors and DRV chip to allow more packed designs
Parts:
- C51: footprint RS485-tester-STM32F405RG.place.kicad:CAPC3216X160 -> BLDC:CAPC3216X160
- D0, D2: footprint RS485-tester-STM32F405RG.place.kicad:LEDSC16080X80 -> BLDC:LEDSC16080X80
- D3: footprint RS485-tester-STM32F405RG.place.kicad:rhom-SMLP34RGB-fp -> BLDC:rhom-SMLP34RGB-fp
- H0, H1, H2, H3: footprint RS485-tester-STM32F405RG.place.kicad:mounting-hole-pkg -> BLDC:mounting-hole-pkg
- J1, J4: footprint RS485-tester-STM32F405RG.place.kicad:molex-microfit-5-pkg -> BLDC:molex-microfit-5-pkg
- J2: footprint RS485-tester-STM32F405RG.place.kicad:molex-microfit-3-pkg_242 -> BLDC:molex-microfit-3-pkg_242
- J3: footprint RS485-tester-STM32F405RG.place.kicad:TC2030-MCP-NL-pkg -> BLDC:TC2030-MCP-NL-pkg
- S1: footprint RS485-tester-STM32F405RG.place.kicad:SW_B3U-1000P -> BLDC:SW_B3U-1000P
- U0: footprint RS485-tester-STM32F405RG.place.kicad:LGA-14L -> BLDC:LGA-14L
- U12: footprint RS485-tester-STM32F405RG.place.kicad:MSOP-8 -> BLDC:MSOP-8
- U3, U7: footprint RS485-tester-STM32F405RG.place.kicad:SOT95P280X145-5N -> BLDC:SOT95P280X145-5N
- U5: footprint RS485-tester-STM32F405RG.place.kicad:HTSSOP-44 -> BLDC:HTSSOP-44
- U6: footprint RS485-tester-STM32F405RG.place.kicad:SOIC127PO650X300-8N -> BLDC:SOIC127PO650X300-8N
- XTAL0: footprint RS485-tester-STM32F405RG.place.kicad:ABM7-8MHZ-D2Y-T-pkg -> BLDC:ABM7-8MHZ-D2Y-T-pkg
Changed lines of the file:
@@
 F 0 "J4" H 6300 5800 40  0000 C CNN
 F 1 "436500513" H 6000 6500 40  0000 C CNN
-F 2 "RS485-tester-STM32F405RG.place.kicad:molex-microfit-5-pkg" H 6200 6200 60  0001 C CNN
+F 2 "BLDC:molex-microfit-5-pkg" H 6200 6200 60  0001 C CNN
 F 3 "" H 6200 6200 60  0001 C CNN
 	1    6200 6150
@@
 F 0 "J2" H 6250 4200 40  0000 C CNN
 F 1 "436500313" H 5850 3700 40  0000 C CNN
-F 2 "RS485-tester-STM32F405RG.place.kicad:molex-microfit-3-pkg_242" H 6050 3950 60  0001 C CNN
+F 2 "BLDC:molex-microfit-3-pkg_242" H 6050 3950 60  0001 C CNN
 F 3 "" H 6050 3950 60  0001 C CNN
 	1    6050 3950
@@
 F 0 "J1" H 5050 5800 40  0000 C CNN
 F 1 "436500513" H 4700 6500 40  0000 C CNN
-F 2 "RS485-tester-STM32F405RG.place.kicad:molex-microfit-5-pkg" H 4900 6200 60  0001 C CNN
+F 2 "BLDC:molex-microfit-5-pkg" H 4900 6200 60  0001 C CNN
 F 3 "" H 4900 6200 60  0001 C CNN
 	1    4900 6150
@@
 F 0 "U12" H 2900 9500 28  0000 L CNN
 F 1 "MCP9808" H 2750 9750 28  0000 L CNN
-F 2 "RS485-tester-STM32F405RG.place.kicad:MSOP-8" H 2850 9750 60  0001 C CNN
+F 2 "BLDC:MSOP-8" H 2850 9750 60  0001 C CNN
 F 3 "" H 2850 9750 60  0001 C CNN
 	1    2850 9750
@@
 F 0 "D3" H 1350 9200 28  0000 L CNN
 F 1 "SMLP34RGB" H 1350 9150 28  0000 L CNN
-F 2 "RS485-tester-STM32F405RG.place.kicad:rhom-SMLP34RGB-fp" H 1600 9000 60  0001 C CNN
+F 2 "BLDC:rhom-SMLP34RGB-fp" H 1600 9000 60  0001 C CNN
 F 3 "" H 1600 9000 60  0001 C CNN
 	1    1600 9000
@@
 F 0 "D2" H 1200 9300 28  0000 L CNN
 F 1 "LTST-C190GKT" V 1150 8850 28  0000 L CNN
-F 2 "RS485-tester-STM32F405RG.place.kicad:LEDSC16080X80" H 1100 9250 60  0001 C CNN
+F 2 "BLDC:LEDSC16080X80" H 1100 9250 60  0001 C CNN
 F 3 "" H 1100 9250 60  0001 C CNN
 	1    1100 9250
@@
 F 0 "C51" H 7750 1300 28  0000 L CNN
 F 1 "2.2μF" H 7750 1350 28  0000 L CNN
-F 2 "RS485-tester-STM32F405RG.place.kicad:CAPC3216X160" H 7650 1350 60  0001 C CNN
+F 2 "BLDC:CAPC3216X160" H 7650 1350 60  0001 C CNN
 F 3 "" H 7650 1350 60  0001 C CNN
 F 4 "2.2uF" H 7650 1350 60  0001 C CNN "Capacitance"
@@
 F 0 "J3" H 8250 5000 28  0000 L CNN
 F 1 "TC2030-MCP-NL" H 8250 5450 28  0000 L CNN
-F 2 "RS485-tester-STM32F405RG.place.kicad:TC2030-MCP-NL-pkg" H 8250 5300 60  0001 C CNN
+F 2 "BLDC:TC2030-MCP-NL-pkg" H 8250 5300 60  0001 C CNN
 F 3 "" H 8250 5300 60  0001 C CNN
 	1    8250 5300
@@
 F 0 "U6" H 5100 5450 28  0000 L CNN
 F 1 "ISL32458E" H 5050 4800 28  0000 L CNN
-F 2 "RS485-tester-STM32F405RG.place.kicad:SOIC127PO650X300-8N" H 5350 5150 60  0001 C CNN
+F 2 "BLDC:SOIC127PO650X300-8N" H 5350 5150 60  0001 C CNN
 F 3 "" H 5350 5150 60  0001 C CNN
 	1    5350 5150
@@
 F 0 "U5" H 3300 4150 28  0000 L CNN
 F 1 "DRV8312" H 3300 4050 28  0000 L CNN
-F 2 "RS485-tester-STM32F405RG.place.kicad:HTSSOP-44" H 3600 2650 60  0001 C CNN
+F 2 "BLDC:HTSSOP-44" H 3600 2650 60  0001 C CNN
 F 3 "" H 3600 2650 60  0001 C CNN
 	1    3600 2650
@@
 F 0 "S1" H 7700 7350 28  0000 L CNN
 F 1 "B3U-1000P" H 7700 7150 28  0000 L CNN
-F 2 "RS485-tester-STM32F405RG.place.kicad:SW_B3U-1000P" H 7800 7250 60  0001 C CNN
+F 2 "BLDC:SW_B3U-1000P" H 7800 7250 60  0001 C CNN
 F 3 "" H 7800 7250 60  0001 C CNN
 	1    7800 7250
@@
 F 0 "H3" H 11550 3975 28  0000 L CNN
 F 1 "NONE" H 11650 3900 60  0001 C CNN
-F 2 "RS485-tester-STM32F405RG.place.kicad:mounting-hole-pkg" H 11650 3900 60  0001 C CNN
+F 2 "BLDC:mounting-hole-pkg" H 11650 3900 60  0001 C CNN
 F 3 "" H 11650 3900 60  0001 C CNN
 	1    11650 3900
@@
 F 0 "U3" H 10450 1550 28  0000 L CNN
 F 1 "TLV702" H 10450 1150 28  0000 L CNN
-F 2 "RS485-tester-STM32F405RG.place.kicad:SOT95P280X145-5N" H 10550 1350 60  0001 C CNN
+F 2 "BLDC:SOT95P280X145-5N" H 10550 1350 60  0001 C CNN
 F 3 "" H 10550 1350 60  0001 C CNN
 	1    10550 1350
@@
 F 0 "H2" H 11550 3525 28  0000 L CNN
 F 1 "NONE" H 11650 3450 60  0001 C CNN
-F 2 "RS485-tester-STM32F405RG.place.kicad:mounting-hole-pkg" H 11650 3450 60  0001 C CNN
+F 2 "BLDC:mounting-hole-pkg" H 11650 3450 60  0001 C CNN
 F 3 "" H 11650 3450 60  0001 C CNN
 	1    11650 3450
@@
 F 0 "H1" H 11550 4425 28  0000 L CNN
 F 1 "NONE" H 11650 4350 60  0001 C CNN
-F 2 "RS485-tester-STM32F405RG.place.kicad:mounting-hole-pkg" H 11650 4350 60  0001 C CNN
+F 2 "BLDC:mounting-hole-pkg" H 11650 4350 60  0001 C CNN
 F 3 "" H 11650 4350 60  0001 C CNN
 	1    11650 4350
@@
 F 0 "U7" H 6350 5400 28  0000 L CNN
 F 1 "SN74LVC1G66DCKR" H 6350 5000 28  0000 L CNN
-F 2 "RS485-tester-STM32F405RG.place.kicad:SOT95P280X145-5N" H 6450 5200 60  0001 C CNN
+F 2 "BLDC:SOT95P280X145-5N" H 6450 5200 60  0001 C CNN
 F 3 "" H 6450 5200 60  0001 C CNN
 	1    6450 5200
@@
 F 0 "XTAL0" H 9050 6450 28  0000 L CNN
 F 1 "ABM7-8.000MHZ-D2Y-T" V 8900 6550 28  0000 L CNN
-F 2 "RS485-tester-STM32F405RG.place.kicad:ABM7-8MHZ-D2Y-T-pkg" H 8950 6450 60  0001 C CNN
+F 2 "BLDC:ABM7-8MHZ-D2Y-T-pkg" H 8950 6450 60  0001 C CNN
 F 3 "" H 8950 6450 60  0001 C CNN
 	1    8950 6450
@@
 F 0 "D0" H 900 9300 28  0000 L CNN
 F 1 "LTST-C190GKT" V 850 8850 28  0000 L CNN
-F 2 "RS485-tester-STM32F405RG.place.kicad:LEDSC16080X80" H 800 9250 60  0001 C CNN
+F 2 "BLDC:LEDSC16080X80" H 800 9250 60  0001 C CNN
 F 3 "" H 800 9250 60  0001 C CNN
 	1    800  9250
@@
 F 0 "U0" H 5100 8150 28  0000 L CNN
 F 1 "LSM6DS3US" H 4950 7450 28  0000 L CNN
-F 2 "RS485-tester-STM32F405RG.place.kicad:LGA-14L" H 4750 7800 60  0001 C CNN
+F 2 "BLDC:LGA-14L" H 4750 7800 60  0001 C CNN
 F 3 "" H 4750 7800 60  0001 C CNN
 	1    4750 7800
@@
 F 0 "H0" H 11550 3125 28  0000 L CNN
 F 1 "NONE" H 11650 3050 60  0001 C CNN
-F 2 "RS485-tester-STM32F405RG.place.kicad:mounting-hole-pkg" H 11650 3050 60  0001 C CNN
+F 2 "BLDC:mounting-hole-pkg" H 11650 3050 60  0001 C CNN
 F 3 "" H 11650 3050 60  0001 C CNN
 	1    11650 3050
