File: BLDC.sch (KiCad schematic (older format))
At the start: 118 parts, among them J1 436500513, J2 436500313, J3 TC2030-MCP-NL, J4 436500513, U0 LSM6DS3US, U12 MCP9808, U13 AS5047D-ATSM, U17 INA250, U18 INA250, U19 INA250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

Commit message: toying with some major layout changes to move the MCU far away from EMI
Parts:
- C51: footprint BLDC:CAPC3216X160 -> Capacitor_SMD:C_1206_3216Metric
- D0, D2: footprint BLDC:LEDSC16080X80 -> Diode_SMD:D_0603_1608Metric
- J1: value 436500513 -> 43650-0510; footprint BLDC:molex-microfit-5-pkg -> BLDC:molex-436500511
- U12: footprint BLDC:MSOP-8 -> Package_SO:MSOP-8_3x3mm_P0.65mm
- U13: value AS5047D-ATSM -> AS5047U; footprint Housings_SSOP:SSOP-14_5.3x6.2mm_Pitch0.65mm -> Package_SO:TSSOP-14_4.4x5mm_P0.65mm
- U3, U7: footprint BLDC:SOT95P280X145-5N -> Package_TO_SOT_SMD:SOT-23-5
- U6: footprint BLDC:SOIC127PO650X300-8N -> Package_SO:SOIC-8_3.9x4.9mm_P1.27mm
Connections:
- net labels removed: ENC_A, ENC_B
- wire segments 492 -> 479
Other:
- note added: "Magnetic Encoder"
- note removed: "Magnetometer"
- moved on the sheet: C39, C60, C62, C66

Commit message: Preliminary routing of new STM position, still to check and refine
Parts:
- removed R30, R31, R33: 39.2kΩ, Resistor_SMD:R_0402_1005Metric, symbol Device:R_Small_US
- removed R38, R43, R47: 2.21kΩ, Resistor_SMD:R_0402_1005Metric, symbol Device:R_Small_US
Connections:
- net labels removed: ENC_MAG_HI, ENC_MAG_LO, ENC_PROG, VSENSE_A, VSENSE_B, VSENSE_C
- wire segments 479 -> 461

Commit message: WIP adding output snubbers and trying to improve high-power paths
Parts:
- removed C66: 1.0μF, Capacitor_SMD:C_0402_1005Metric, symbol Device:C_Small
- added C23, C28: DNP, Capacitor_SMD:C_0603_1608Metric, symbol Device:C_Small
- added R12, R13: DNP, Resistor_SMD:R_0805_2012Metric, symbol Device:R_Small
- C1, C11, C64, C68: footprint Capacitor_SMD:C_0805_2012Metric -> Capacitor_SMD:C_0603_1608Metric
- R7: footprint Resistor_SMD:R_0805_2012Metric -> Resistor_SMD:R_0603_1608Metric
Connections:
- wire segments 461 -> 467
Other:
- note added: "TODO:\nrc snubbers"
- note added: "snubber"
- moved on the sheet: J2
Changed lines of the file:
@@
 Text Label 11950 7150 0    40   ~ 0
 MOT_OCTW
-Text Label 11450 5750 1    40   ~ 0
+Text Label 10250 5750 1    40   ~ 0
 SPI_CS
 Text Label 11950 6950 0    40   ~ 0
@@
 Text Label 2550 9600 2    40   ~ 0
 I2C_SDA
-Text Label 5300 3950 0    40   ~ 0
+Text Label 1150 1650 0    40   ~ 0
 driver_phase-B
-Text Label 5300 4050 0    40   ~ 0
+Text Label 1150 1750 0    40   ~ 0
 driver_phase-C
-Text Label 5300 3850 0    40   ~ 0
+Text Label 1150 1550 0    40   ~ 0
 driver_phase-A
 Text Label 1100 10050 1    40   ~ 0
@@
 	800  9000 1100 9000
 Wire Wire Line
-	5800 3950 5300 3950
+	1650 1650 1150 1650
 Wire Wire Line
-	5800 4050 5300 4050
+	1650 1750 1150 1750
 Wire Wire Line
-	5800 3850 5300 3850
+	1650 1550 1150 1550
 Wire Wire Line
 	7800 6550 7800 6700
@@
 	4000 2400 4250 2400
 Wire Wire Line
-	4000 3800 4550 3800
-Wire Wire Line
-	4000 2900 4550 2900
-Wire Wire Line
 	4000 2100 4550 2100
 Connection ~ 4100 2000
@@
 Connection ~ 4100 3100
 Wire Wire Line
-	5050 3100 4950 3100
-Wire Wire Line
 	4000 3300 4100 3300
 Wire Wire Line
@@
 Connection ~ 4100 3300
 Wire Wire Line
-	5050 3300 4950 3300
+	5150 3300 4950 3300
 Wire Wire Line
 	5050 2400 4950 2400
@@
 Connection ~ 4650 3300
 Wire Wire Line
-	4950 3450 5050 3450
+	4950 3450 5150 3450
 Wire Wire Line
-	5050 3450 5050 3300
+	5150 3450 5150 3300
 Wire Wire Line
 	4000 2300 4450 2300
@@
 	4100 2000 5250 2000
 Wire Wire Line
-	4100 2800 5250 2800
-Wire Wire Line
-	4100 3700 5250 3700
-Wire Wire Line
 	3650 4450 3400 4450
 Wire Wire Line
@@
 DISCO_BUS_OUT
 Connection ~ 10250 8400
-Connection ~ 5050 3450
+Connection ~ 5150 3450
 Connection ~ 5250 9050
 Connection ~ 5250 9950
@@
 Text Label 5250 2000 2    40   ~ 0
 driver_phase-A
-Text Label 5250 2800 2    40   ~ 0
+Text Label 4550 2800 0    40   ~ 0
 driver_phase-B
-Text Label 5250 3700 2    40   ~ 0
+Text Label 4550 3700 0    40   ~ 0
 driver_phase-C
-Text Label 4550 3800 2    40   ~ 0
+Text Label 4550 3800 0    40   ~ 0
 GND_C
-Text Label 4550 2900 0    40   ~ 0
-GND_B
 Text Label 4550 2100 0    40   ~ 0
 GND_A
@@
 L power:GND #PWR092
 U 1 1 5BCC8183
-P 6100 4250
-F 0 "#PWR092" H 6100 4000 50  0001 C CNN
-F 1 "GND" H 6100 4100 50  0000 C CNN
-F 2 "" H 6100 4250 50  0001 C CNN
-F 3 "" H 6100 4250 50  0001 C CNN
-	1    6100 4250
+P 1950 1950
+F 0 "#PWR092" H 1950 1700 50  0001 C CNN
+F 1 "GND" H 1950 1800 50  0001 C CNN
+F 2 "" H 1950 1950 50  0001 C CNN
+F 3 "" H 1950 1950 50  0001 C CNN
+	1    1950 1950
 	1    0    0    -1
 $EndComp
 $Comp
-L power:GND #PWR091
-U 1 1 5BCC7F9B
-P 6100 3650
-F 0 "#PWR091" H 6100 3400 50  0001 C CNN
-F 1 "GND" H 6100 3500 50  0000 C CNN
-F 2 "" H 6100 3650 50  0001 C CNN
-F 3 "" H 6100 3650 50  0001 C CNN
-	1    6100 3650
-	-1   0    0    1
-$EndComp
-$Comp
 L power:GND #PWR089
 U 1 1 5BCBFE31
@@
 L BLDC:generic-box-sym$2 J2
 U 1 1 5BCA5BD2
-P 6050 3950
-F 0 "J2" H 6250 4200 40  0000 C CNN
-F 1 "436500313" H 5850 3700 40  0000 C CNN
-F 2 "BLDC:molex-microfit-3-pkg_242" H 6050 3950 60  0001 C CNN
-F 3 "" H 6050 3950 60  0001 C CNN
-	1    6050 3950
+P 1900 1650
+F 0 "J2" H 1750 1900 40  0000 C CNN
+F 1 "436500313" H 1700 1400 40  0000 C CNN
+F 2 "BLDC:molex-microfit-3-pkg_242" H 1900 1650 60  0001 C CNN
+F 3 "" H 1900 1650 60  0001 C CNN
+	1    1900 1650
 	1    0    0    -1
 $EndComp
@@
 P 10550 1850
 F 0 "#PWR073" H 10550 1600 50  0001 C CNN
-F 1 "GND" H 10550 1700 50  0000 C CNN
+F 1 "GND" H 10550 1700 50  0001 C CNN
 F 2 "" H 10550 1850 50  0001 C CNN
 F 3 "" H 10550 1850 50  0001 C CNN
@@
 P 1600 3650
 F 0 "#PWR059" H 1600 3400 50  0001 C CNN
-F 1 "GND" H 1600 3500 50  0000 C CNN
+F 1 "GND" H 1600 3500 50  0001 C CNN
 F 2 "" H 1600 3650 50  0001 C CNN
 F 3 "" H 1600 3650 50  0001 C CNN
@@
 $EndComp
 $Comp
-L power:GND #PWR056
-U 1 1 5B54BD24
-P 5050 3100
-F 0 "#PWR056" H 5050 2850 50  0001 C CNN
-F 1 "GND" H 5050 2950 50  0000 C CNN
-F 2 "" H 5050 3100 50  0001 C CNN
-F 3 "" H 5050 3100 50  0001 C CNN
-	1    5050 3100
-	0    -1   -1   0
-$EndComp
-$Comp
 L power:GND #PWR055
 U 1 1 5B54BB36
-P 5050 3450
-F 0 "#PWR055" H 5050 3200 50  0001 C CNN
-F 1 "GND" H 5050 3300 50  0000 C CNN
-F 2 "" H 5050 3450 50  0001 C CNN
-F 3 "" H 5050 3450 50  0001 C CNN
-	1    5050 3450
-	0    -1   -1   0
+P 5150 3450
+F 0 "#PWR055" H 5150 3200 50  0001 C CNN
+F 1 "GND" H 5150 3300 50  0001 C CNN
+F 2 "" H 5150 3450 50  0001 C CNN
+F 3 "" H 5150 3450 50  0001 C CNN
+	1    5150 3450
+	1    0    0    -1
 $EndComp
 $Comp
@@
 P 8400 2450
 F 0 "#PWR041" H 8400 2200 50  0001 C CNN
-F 1 "GND" H 8400 2300 50  0000 C CNN
+F 1 "GND" H 8400 2300 50  0001 C CNN
 F 2 "" H 8400 2450 50  0001 C CNN
 F 3 "" H 8400 2450 50  0001 C CNN
@@
 F 0 "C68" V 4650 2150 28  0000 L CNN
 F 1 "100.0nF" V 4650 2350 28  0000 L CNN
-F 2 "Capacitor_SMD:C_0805_2012Metric" H 4700 2300 60  0001 C CNN
+F 2 "Capacitor_SMD:C_0603_1608Metric" H 4700 2300 60  0001 C CNN
 F 3 "" H 4700 2300 60  0001 C CNN
 F 4 "0.1uF" H 4700 2300 60  0001 C CNN "Capacitance"
@@
 $EndComp
 $Comp
-L Device:C_Small C66
-U 1 1 5B48C3EF
-P 4300 9450
-F 0 "C66" H 4400 9400 28  0000 L CNN
-F 1 "1.0μF" H 4400 9450 28  0000 L CNN
-F 2 "Capacitor_SMD:C_0402_1005Metric" H 4300 9450 60  0001 C CNN
-F 3 "" H 4300 9450 60  0001 C CNN
-F 4 "1.0uF" H 4300 9450 60  0001 C CNN "Capacitance"
-F 5 "40.0%" H 4300 9450 60  0001 C CNN "Tolerance"
-F 6 "25.0V" H 4400 9500 28  0000 L CNN "Maximum Voltage"
-	1    4300 9450
-	-1   0    0    1
-$EndComp
-$Comp
 L Device:R_Small_US R50
 U 1 1 5B48C3ED
@@
 F 0 "C64" V 4800 2950 28  0000 L CNN
 F 1 "100.0nF" V 4800 3150 28  0000 L CNN
-F 2 "Capacitor_SMD:C_0805_2012Metric" H 4850 3100 60  0001 C CNN
+F 2 "Capacitor_SMD:C_0603_1608Metric" H 4850 3100 60  0001 C CNN
 F 3 "" H 4850 3100 60  0001 C CNN
 F 4 "0.1uF" H 4850 3100 60  0001 C CNN "Capacitance"
@@
 P 7650 1500
 F 0 "#PWR040" H 7650 1250 50  0001 C CNN
-F 1 "GND" H 7650 1350 50  0000 C CNN
+F 1 "GND" H 7650 1350 50  0001 C CNN
 F 2 "" H 7650 1500 50  0001 C CNN
 F 3 "" H 7650 1500 50  0001 C CNN
@@
 P 7700 4250
 F 0 "#PWR0110" H 7700 4000 50  0001 C CNN
-F 1 "GND" H 7700 4100 50  0000 C CNN
+F 1 "GND" H 7700 4100 50  0001 C CNN
 F 2 "" H 7700 4250 50  0001 C CNN
 F 3 "" H 7700 4250 50  0001 C CNN
@@
 P 6950 3300
 F 0 "#PWR0111" H 6950 3050 50  0001 C CNN
-F 1 "GND" H 6950 3150 50  0000 C CNN
+F 1 "GND" H 6950 3150 50  0001 C CNN
 F 2 "" H 6950 3300 50  0001 C CNN
 F 3 "" H 6950 3300 50  0001 C CNN
@@
 F 0 "R7" H 8050 3300 28  0000 L CNN
 F 1 "8.87MΩ" H 8050 3250 28  0000 L CNN
-F 2 "Resistor_SMD:R_0805_2012Metric" H 8000 3300 60  0001 C CNN
+F 2 "Resistor_SMD:R_0603_1608Metric" H 8000 3300 60  0001 C CNN
 F 3 "" H 8000 3300 60  0001 C CNN
 F 4 "8870000.0ohm" H 8000 3300 60  0001 C CNN "Resistance"
@@
 F 0 "C11" H 8200 3250 28  0000 L CNN
 F 1 "150pF" H 8150 3300 28  0000 L CNN
-F 2 "Capacitor_SMD:C_0805_2012Metric" H 8400 3300 60  0001 C CNN
+F 2 "Capacitor_SMD:C_0603_1608Metric" H 8400 3300 60  0001 C CNN
 F 3 "" H 8400 3300 60  0001 C CNN
 F 4 "150pF" H 8400 3300 60  0001 C CNN "Capacitance"
@@
 F 0 "C1" V 4650 1400 28  0000 L CNN
 F 1 "100.0nF" V 4650 1550 28  0000 L CNN
-F 2 "Capacitor_SMD:C_0805_2012Metric" H 4700 1500 60  0001 C CNN
+F 2 "Capacitor_SMD:C_0603_1608Metric" H 4700 1500 60  0001 C CNN
 F 3 "" H 4700 1500 60  0001 C CNN
 F 4 "0.1uF" H 4700 1500 60  0001 C CNN "Capacitance"
@@
 $EndComp
 Connection ~ 3000 1100
-Connection ~ 3950 9350
-Wire Wire Line
-	3950 9350 4300 9350
-Wire Wire Line
-	3950 9550 4300 9550
-Connection ~ 3950 9550
 $Comp
 L Device:R_Small_US R9
@@
 	11250 8500 11350 8500
 Connection ~ 11350 8500
+Text Notes 5450 2000 0    79   ~ 16
+TODO:\nrc snubbers
+Wire Wire Line
+	1950 1350 2150 1350
+Wire Wire Line
+	2150 1350 2150 1950
+Wire Wire Line
+	2150 1950 1950 1950
+Connection ~ 1950 1950
+$Comp
+L Device:C_Small C23
+U 1 1 5D6FD1A8
+P 5500 4000
+F 0 "C23" H 5592 4046 50  0000 L CNN
+F 1 "DNP" H 5592 3955 50  0000 L CNN
+F 2 "Capacitor_SMD:C_0603_1608Metric" H 5500 4000 50  0001 C CNN
+F 3 "~" H 5500 4000 50  0001 C CNN
+	1    5500 4000
+	1    0    0    -1
+$EndComp
+$Comp
+L Device:R_Small R12
+U 1 1 5D6FCF61
+P 5500 3800
+F 0 "R12" H 5559 3846 50  0000 L CNN
+F 1 "DNP" H 5559 3755 50  0000 L CNN
+F 2 "Resistor_SMD:R_0805_2012Metric" H 5500 3800 50  0001 C CNN
+F 3 "~" H 5500 3800 50  0001 C CNN
+	1    5500 3800
+	1    0    0    -1
+$EndComp
+Wire Wire Line
+	5350 3800 5350 4100
+Wire Wire Line
+	5350 4100 5500 4100
+Wire Wire Line
+	4000 3800 5350 3800
+Wire Wire Line
+	4100 3700 5500 3700
+Text Notes 5750 3950 0    79   ~ 16
+snubber
+$Comp
+L Device:C_Small C28
+U 1 1 5D918C4F
+P 5500 3100
+F 0 "C28" H 5592 3146 50  0000 L CNN
+F 1 "DNP" H 5592 3055 50  0000 L CNN
+F 2 "Capacitor_SMD:C_0603_1608Metric" H 5500 3100 50  0001 C CNN
+F 3 "~" H 5500 3100 50  0001 C CNN
+	1    5500 3100
+	1    0    0    -1
+$EndComp
+$Comp
+L Device:R_Small R13
+U 1 1 5D918C50
+P 5500 2900
+F 0 "R13" H 5559 2946 50  0000 L CNN
+F 1 "DNP" H 5559 2855 50  0000 L CNN
+F 2 "Resistor_SMD:R_0805_2012Metric" H 5500 2900 50  0001 C CNN
+F 3 "~" H 5500 2900 50  0001 C CNN
+	1    5500 2900
+	1    0    0    -1
+$EndComp
+Wire Wire Line
+	5150 3300 5150 3100
+Wire Wire Line
+	4950 3100 5150 3100
+Connection ~ 5150 3300
+Wire Wire Line
+	5350 2900 5350 3200
+Wire Wire Line
+	5350 3200 5500 3200
+Wire Wire Line
+	4000 2900 5350 2900
+Wire Wire Line
+	4100 2800 5500 2800
+Text Label 4550 2900 0    40   ~ 0
+GND_B
 $EndSCHEMATC

Commit message: finish draft of high-power net routes. clean up throughout.
Parts:
- added C29: DNP, Capacitor_SMD:C_0603_1608Metric, symbol Device:C_Small
- added R14: DNP, Resistor_SMD:R_0805_2012Metric, symbol Device:R_Small
- J4: value 436500513 -> 43650-0510; footprint BLDC:molex-microfit-5-pkg -> BLDC:molex-436500511
Other:
- note removed: "TODO:\nrc snubbers"
Changed lines of the file:
@@
 Wire Wire Line
 	4000 2400 4250 2400
-Wire Wire Line
-	4000 2100 4550 2100
 Connection ~ 4100 2000
 Connection ~ 4100 2800
@@
 	5150 3300 4950 3300
 Wire Wire Line
-	5050 2400 4950 2400
+	5150 2400 4950 2400
 Wire Wire Line
 	4750 3450 4650 3450
@@
 	4000 1600 4250 1600
 Wire Wire Line
-	4800 2300 5050 2300
+	4800 2300 5150 2300
 Wire Wire Line
 	3600 1100 3600 1200
@@
 Connection ~ 4450 3100
 Wire Wire Line
-	5150 2350 5050 2350
-Wire Wire Line
-	5050 2300 5050 2350
-Connection ~ 5050 2350
-Wire Wire Line
 	4650 6050 4600 6050
 Wire Wire Line
@@
 	2900 4150 3100 4150
 Wire Wire Line
-	4100 2000 5250 2000
-Wire Wire Line
 	3650 4450 3400 4450
 Wire Wire Line
@@
 	4450 3100 4750 3100
 Wire Wire Line
-	5050 2350 5050 2400
-Wire Wire Line
 	3800 4250 3800 4450
 Wire Wire Line
@@
 Wire Wire Line
 	2250 5750 1950 5750
-Text Label 5250 2000 2    40   ~ 0
+Text Label 4550 2000 0    40   ~ 0
 driver_phase-A
 Text Label 4550 2800 0    40   ~ 0
@@
 $EndComp
 $Comp
-L power:GND #PWR089
-U 1 1 5BCBFE31
-P 6250 6550
-F 0 "#PWR089" H 6250 6300 50  0001 C CNN
-F 1 "GND" H 6250 6400 50  0000 C CNN
-F 2 "" H 6250 6550 50  0001 C CNN
-F 3 "" H 6250 6550 50  0001 C CNN
-	1    6250 6550
-	1    0    0    -1
-$EndComp
-$Comp
-L power:GND #PWR088
-U 1 1 5BCBFC3D
-P 6250 5750
-F 0 "#PWR088" H 6250 5500 50  0001 C CNN
-F 1 "GND" H 6250 5600 50  0000 C CNN
-F 2 "" H 6250 5750 50  0001 C CNN
-F 3 "" H 6250 5750 50  0001 C CNN
-	1    6250 5750
-	-1   0    0    1
-$EndComp
-$Comp
 L power:+48V #PWR075
 U 1 1 5BCAE07C
@@
 P 6200 6150
 F 0 "J4" H 6300 5800 40  0000 C CNN
-F 1 "436500513" H 6000 6500 40  0000 C CNN
-F 2 "BLDC:molex-microfit-5-pkg" H 6200 6200 60  0001 C CNN
+F 1 "43650-0510" H 6000 6500 40  0000 C CNN
+F 2 "BLDC:molex-436500511" H 6200 6200 60  0001 C CNN
 F 3 "" H 6200 6200 60  0001 C CNN
 	1    6200 6150
@@
 L power:GND #PWR057
 U 1 1 5B54C2E4
-P 5150 2350
-F 0 "#PWR057" H 5150 2100 50  0001 C CNN
-F 1 "GND" H 5150 2200 50  0000 C CNN
-F 2 "" H 5150 2350 50  0001 C CNN
-F 3 "" H 5150 2350 50  0001 C CNN
-	1    5150 2350
-	0    -1   -1   0
+P 5150 2400
+F 0 "#PWR057" H 5150 2150 50  0001 C CNN
+F 1 "GND" H 5150 2250 50  0001 C CNN
+F 2 "" H 5150 2400 50  0001 C CNN
+F 3 "" H 5150 2400 50  0001 C CNN
+	1    5150 2400
+	1    0    0    -1
 $EndComp
 $Comp
@@
 	11250 8500 11350 8500
 Connection ~ 11350 8500
-Text Notes 5450 2000 0    79   ~ 16
-TODO:\nrc snubbers
 Wire Wire Line
 	1950 1350 2150 1350
@@
 Text Label 4550 2900 0    40   ~ 0
 GND_B
+Text Notes 5750 3000 0    79   ~ 16
+snubber
+$Comp
+L Device:C_Small C29
+U 1 1 5D504D64
+P 5500 2300
+F 0 "C29" H 5592 2346 50  0000 L CNN
+F 1 "DNP" H 5592 2255 50  0000 L CNN
+F 2 "Capacitor_SMD:C_0603_1608Metric" H 5500 2300 50  0001 C CNN
+F 3 "~" H 5500 2300 50  0001 C CNN
+	1    5500 2300
+	1    0    0    -1
+$EndComp
+$Comp
+L Device:R_Small R14
+U 1 1 5D504D65
+P 5500 2100
+F 0 "R14" H 5559 2146 50  0000 L CNN
+F 1 "DNP" H 5559 2055 50  0000 L CNN
+F 2 "Resistor_SMD:R_0805_2012Metric" H 5500 2100 50  0001 C CNN
+F 3 "~" H 5500 2100 50  0001 C CNN
+	1    5500 2100
+	1    0    0    -1
+$EndComp
+Wire Wire Line
+	5150 2300 5150 2400
+Connection ~ 5150 2400
+Wire Wire Line
+	4100 2000 5500 2000
+Wire Wire Line
+	5500 2400 5350 2400
+Wire Wire Line
+	5350 2400 5350 2100
+Wire Wire Line
+	4000 2100 5350 2100
 $EndSCHEMATC

Commit message: WIP simplify power supply designs
Parts:
- removed R1: 196.0kΩ, Resistor_SMD:R_0402_1005Metric, symbol Device:R_Small_US
- removed R11: 124.0kΩ, Resistor_SMD:R_0402_1005Metric, symbol Device:R_Small_US
- removed R7: 8.87MΩ, Resistor_SMD:R_0603_1608Metric, symbol Device:R_Small_US
- removed R8: 1.1MΩ, Resistor_SMD:R_0402_1005Metric, symbol Device:R_Small_US
- removed U4: LM5166, Package_SON:VSON-10-1EP_3x3mm_P0.5mm_EP1.65x2.4mm_ThermalVias, symbol BLDC:ti-LM5166
- added R1: 100k, Resistor_SMD:R_0402_1005Metric, symbol Device:R_Small
- added R11: 49k9, Resistor_SMD:R_0603_1608Metric, symbol Device:R_Small
- added R7: 226k, Resistor_SMD:R_0603_1608Metric, symbol Device:R_Small
- added R8: 453k, Resistor_SMD:R_0603_1608Metric, symbol Device:R_Small
- added U4: LM5163, Package_SO:SOIC-8-1EP_3.9x4.9mm_P1.27mm_EP2.41x3.3mm, symbol BLDC:ti-LM5163
- C10: value 4.1pF -> 56p; Maximum Voltage 6.3V -> 50V
- C11: value 150pF -> 3n3; Maximum Voltage 6.3V -> 16V
- C12: value 4.7μF -> 22u; footprint Capacitor_SMD:C_0805_2012Metric -> Capacitor_SMD:C_1210_3225Metric
- C17: value 4.7μF -> 2n2; footprint Capacitor_SMD:C_0805_2012Metric -> Capacitor_SMD:C_0402_1005Metric; Capacitance 4.7μF -> (none); Maximum Voltage 16.0V -> (none); Tolerance 40.0% -> (none)
- C4: value 2.2μF -> 2u2; Maximum Voltage 100.0V -> 100V
- C8: value 56.0nF -> 2u2; footprint Capacitor_SMD:C_0402_1005Metric -> Capacitor_SMD:C_1210_3225Metric; Capacitance 0.056uF -> 2.2uF; Maximum Voltage 16.0V -> 100V
- L2: value 220μH -> 150 uH; footprint Inductor_SMD:L_6.3x6.3_H3 -> Inductor_SMD:L_12x12mm_H6mm
Connections:
- wire segments 467 -> 447
- no-connect marks 0 -> 1
Other:
- note added: "TODO: replace 3v9 supply with LMZ21700SILT"
- note added: "TODO: update with component choices for smaller inductor"
- moved on the sheet: C10, C11, C12, C4, L2

Commit message: Finished simplified power rail design
Parts:
- removed C37: 56.0nF, Capacitor_SMD:C_0402_1005Metric, symbol Device:C_Small
- removed C4, C8: 2u2, Capacitor_SMD:C_1210_3225Metric, symbol Device:C_Small
- removed C51: 2.2μF, Capacitor_SMD:C_1206_3216Metric, symbol Device:C_Small
- removed C58, C6, C7: 100.0μF, Capacitor_SMD:C_1206_3216Metric, symbol Device:C_Small
- removed L0: 22.0μH, Inductor_SMD:L_7.3x7.3_H4.5, symbol BLDC:inductor-sym
- removed R25: 271.0kΩ, Resistor_SMD:R_0402_1005Metric, symbol Device:R_Small_US
- removed R5: 124.0kΩ, Resistor_SMD:R_0402_1005Metric, symbol Device:R_Small_US
- removed U2: LM5166, Package_SON:VSON-10-1EP_3x3mm_P0.5mm_EP1.65x2.4mm_ThermalVias, symbol BLDC:ti-LM5166
- added C31: 22μF, Capacitor_SMD:C_1812_4532Metric, symbol Device:C_Small
- added C34: 3.3nF, Capacitor_SMD:C_0805_2012Metric, symbol Device:C_Small
- added C41: 47.0μF, Capacitor_SMD:C_1206_3216Metric, symbol Device:C_Small
- added C45: 2u2, Capacitor_SMD:C_1210_3225Metric, symbol Device:C_Small
- added R16: 681.0kΩ, Resistor_SMD:R_0402_1005Metric, symbol Device:R_Small_US
- added R17: 180.0kΩ, Resistor_SMD:R_0402_1005Metric, symbol Device:R_Small_US
- added U1: LMZ21700SILT, BLDC:SIL0008E, symbol BLDC:LMZ21700SILT
- C10: value 56p -> 47p; Capacitance 4.1pF -> 47pF
- C11: value 3n3 -> 2n2; footprint Capacitor_SMD:C_0603_1608Metric -> Capacitor_SMD:C_0805_2012Metric; Capacitance 150pF -> 2.2nF; Maximum Voltage 16V -> 50V
- C12: value 22u -> 4.7u; footprint Capacitor_SMD:C_1210_3225Metric -> Capacitor_SMD:C_1206_3216Metric; Maximum Voltage 16.0V -> 25.0V
- C13, C14, C16: footprint Capacitor_SMD:C_0603_1608Metric -> Capacitor_SMD:C_0402_1005Metric
- C17: footprint Capacitor_SMD:C_0402_1005Metric -> Capacitor_SMD:C_0805_2012Metric
- L2: value 150 uH -> 100 uH
- R7: value 226k -> 237k
Connections:
- net labels removed: MOT_PWR_EN
- wire segments 447 -> 425
- no-connect marks 1 -> 2
Other:
- moved on the sheet: R1

Commit message: switch to larger accel package. enlarge all vias and traces. clean up.
Parts:
- removed U0: LSM6DS3US, BLDC:LGA-14L, symbol BLDC:st-LSM6DS3US
- added C4, C6: 4u7, Capacitor_SMD:C_1210_3225Metric, symbol Device:C_Small
- added U2: IIS328DQ, Package_DFN_QFN:QFN-24-1EP_4x4mm_P0.5mm_EP2.6x2.6mm, symbol BLDC:IIS328DQ
- C45: value 2u2 -> 4u7; Capacitance 2.2uF -> (none); D1N (none) -> Digikey; D1PN (none) -> 1276-7060-1-ND; MFN (none) -> Samsung; MPN (none) -> CL32B475KCVZW6E; Tolerance 40.0% -> 10%
- L2: value 100 uH -> 82 uH; footprint Inductor_SMD:L_12x12mm_H6mm -> Inductor_SMD:L_7.3x7.3_H4.5; D1N (none) -> Digikey; D1PN (none) -> 513-1666-1-ND; MFN (none) -> Eaton; MPN (none) -> DR74-820-R
- R1: value 100k -> 40k2
- R7: value 237k -> 255k
- U1: value LMZ21700SILT -> LMZ21700SIL
- renumbered XTAL0 to X0
Connections:
- no-connect marks 2 -> 20
Other:
- note added: "1.6ms\nsoft-start time"
- note added: "TODO: draw this nicer"
- note added: "top-side ceramics"
- note removed: "TODO: replace 3v9 supply with LMZ21700SILT"
- note removed: "TODO: update with component choices for smaller inductor"
- moved on the sheet: C2, C20, C21, C25, C3, C31, C34, C35, C41, C5, C62, C9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

Commit message: use NRST for SWD_RESET
Connections:
- wire segments 425 -> 424
Changed lines of the file:
@@
 Text Label 11950 6950 0    40   ~ 0
 MOT_RST_A
-Text Label 10650 7650 3    40   ~ 0
+Text Label 9750 6550 2    40   ~ 0
 SWD_RESET
 Text Label 11950 6150 0    40   ~ 0
@@
 Wire Wire Line
 	8270 2100 8275 2100
-Wire Wire Line
-	8275 2100 8725 2100
 Connection ~ 8725 2100
 Wire Wire Line
