File: BLDC.sch (KiCad schematic (older format))
At the start: 122 parts, among them J1 43650-0510, J2 436500313, J3 DNP, J4 43650-0510, J5 BONUS, U1 LMZ21700SIL, U10 INA253, U11 INA253, U12 MCP9808, U13 AS5047U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

Commit message: Added 3d model for regulator, routed all design (passing DRC)
Parts:
- C10, C8: footprint Capacitor_SMD:C_0603_1608Metric -> Capacitor_SMD:C_0402_1005Metric
Changed lines of the file:
@@
 F 0 "C10" H 8075 2825 39  0000 L CNN
 F 1 "2u2" H 8075 2750 39  0000 L CNN
-F 2 "Capacitor_SMD:C_0603_1608Metric" H 8300 2800 60  0001 C CNN
+F 2 "Capacitor_SMD:C_0402_1005Metric" H 8300 2800 60  0001 C CNN
 F 3 "~" H 8300 2800 60  0001 C CNN
 F 4 "2.2uF" H 8300 2800 60  0001 C CNN "Capacitance"
@@
 F 0 "C8" H 8875 3975 39  0000 L CNN
 F 1 "2u2" H 8875 3900 39  0000 L CNN
-F 2 "Capacitor_SMD:C_0603_1608Metric" H 9100 3950 60  0001 C CNN
+F 2 "Capacitor_SMD:C_0402_1005Metric" H 9100 3950 60  0001 C CNN
 F 3 "~" H 9100 3950 60  0001 C CNN
 F 4 "2.2uF" H 9100 3950 60  0001 C CNN "Capacitance"

Commit message: place/route tweaks. move accelerometer to top layer.
Parts:
- D0, D2: symbol BLDC:diode-sym$2 -> Device:LED_Small
- L2: D1PN 513-1666-1-ND -> 732-1199; MFN Eaton -> Wurth; MPN CHANGEME -> 744777920
Changed lines of the file:
@@
 $EndComp
 $Comp
-L BLDC:diode-sym$2 D2
+L Device:LED_Small D2
 U 1 1 5B48C3C8
 P 1100 9250
@@
 F 7 "LTST-C190GKT" H 1200 9400 50  0001 C CNN "MPN"
 	1    1100 9250
-	1    0    0    -1
+	0    -1   -1   0
 $EndComp
 $Comp
@@
 $EndComp
 $Comp
-L BLDC:diode-sym$2 D0
+L Device:LED_Small D0
 U 1 1 5B48C40B
 P 800 9250
@@
 F 7 "LTST-C190GKT" H 900 9400 50  0001 C CNN "MPN"
 	1    800  9250
-	1    0    0    -1
+	0    -1   -1   0
 $EndComp
 $Comp
@@
 F 3 "" H 8850 3450 60  0001 C CNN
 F 4 "Digikey" V 8850 3450 50  0001 C CNN "D1N"
-F 5 "513-1666-1-ND" V 8850 3450 50  0001 C CNN "D1PN"
+F 5 "732-1199" V 8850 3450 50  0001 C CNN "D1PN"
 F 6 "100.0uH" H 8850 3450 60  0001 C CNN "Inductance"
-F 7 "Eaton" V 8850 3450 50  0001 C CNN "MFN"
-F 8 "CHANGEME" V 8850 3450 50  0001 C CNN "MPN"
+F 7 "Wurth" V 8850 3450 50  0001 C CNN "MFN"
+F 8 "744777920" V 8850 3450 50  0001 C CNN "MPN"
 F 9 "1A" H 8850 3450 60  0001 C CNN "Maximum Current"
 F 10 "20%" H 8850 3450 60  0001 C CNN "Tolerance"
