File: BLDC.kicad_sch (KiCad schematic)
At the start: 124 parts, among them J1 43650-0510, J2 436500313, J3 DNP, J4 43650-0510, J5 BONUS, U1 LMZ21700SIL, U10 INA253, U11 INA253, U12 MCP9808, U13 AS5047U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

Commit message: Correcting voltage divider
Parts:
- R3: value 59k -> 47.5k; D1PN 311-59KLRCT-ND -> 311-47.5KLRCT-ND; MPN RC0402FR-0759KL -> RC0402FR-0747K5L; Resistance 59000.0ohm -> 47500.0ohm
Other:
- note added: "Enable at 2.1V Ven = 2.1*5.75 = 12.075V"
- note removed: "Enable at 2.1V Ven = 2.1*59/10 = 12.39V"
Changed lines of the file:
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@@
   (junction (at 331.47 151.13))
   (junction (at 331.47 158.75))
-  (no_connect (at 199.517 85.09))
   (no_connect (at 206.375 48.26))
-  (no_connect (at 182.499 229.108))
-  (no_connect (at 182.499 239.268))
+  (no_connect (at 137.16 240.03))
+  (no_connect (at 137.16 245.11))
   (no_connect (at 182.499 246.888))
-  (no_connect (at 206.629 259.588))
-  (no_connect (at 182.499 244.348))
+  (no_connect (at 137.16 247.65))
+  (no_connect (at 199.517 95.25))
+  (no_connect (at 182.499 249.428))
   (no_connect (at 137.16 237.49))
-  (no_connect (at 137.16 242.57))
   (no_connect (at 182.499 251.968))
+  (no_connect (at 206.629 259.588))
+  (no_connect (at 137.16 242.57))
+  (no_connect (at 182.499 239.268))
   (no_connect (at 219.837 95.25))
-  (no_connect (at 182.499 241.808))
-  (no_connect (at 182.499 249.428))
+  (no_connect (at 182.499 244.348))
   (no_connect (at 182.499 234.188))
-  (no_connect (at 182.499 236.728))
-  (no_connect (at 137.16 247.65))
+  (no_connect (at 199.517 85.09))
+  (no_connect (at 137.16 234.95))
+  (no_connect (at 182.499 229.108))
   (no_connect (at 247.396 40.64))
-  (no_connect (at 137.16 245.11))
-  (no_connect (at 137.16 240.03))
   (no_connect (at 182.499 231.648))
-  (no_connect (at 137.16 234.95))
-  (no_connect (at 199.517 95.25))
+  (no_connect (at 182.499 241.808))
+  (no_connect (at 182.499 236.728))
   (wire (pts (xy 19.685 72.39) (xy 26.035 72.39))
     (stroke (width 0) (type solid) (color 0 0 0 0))
@@
     (effects (font (size 2.54 2.54)) (justify left bottom))
   )
-  (text "Enable at 2.1V\nVen = 2.1*59/10 = 12.39V" (at 196.596 100.076 180)
+  (text "Enable at 2.1V\nVen = 2.1*5.75 = 12.075V" (at 196.596 100.076 180)
     (effects (font (size 1.27 1.27)) (justify right bottom))
   )
@@
       (effects (font (size 0.9906 0.9906)) (justify left))
     )
-    (property "Value" "59k" (id 1) (at 193.675 78.994 0)
+    (property "Value" "47.5k" (id 1) (at 193.675 78.994 0)
       (effects (font (size 0.9906 0.9906)) (justify left))
     )
@@
       (effects (font (size 1.27 1.27)) hide)
     )
-    (property "D1PN" "311-59KLRCT-ND" (id 5) (at 193.548 82.042 0)
+    (property "D1PN" "311-47.5KLRCT-ND" (id 5) (at 193.548 82.042 0)
       (effects (font (size 1.27 1.27)) hide)
     )
@@
       (effects (font (size 1.27 1.27)) hide)
     )
-    (property "MPN" "RC0402FR-0759KL" (id 7) (at 193.548 82.042 0)
+    (property "MPN" "RC0402FR-0747K5L" (id 7) (at 193.548 82.042 0)
       (effects (font (size 1.27 1.27)) hide)
     )
@@
       (effects (font (size 1.524 1.524)) hide)
     )
-    (property "Resistance" "59000.0ohm" (id 9) (at 194.818 79.502 0)
+    (property "Resistance" "47500.0ohm" (id 9) (at 194.818 79.502 0)
       (effects (font (size 1.524 1.524)) hide)
     )
